File: schematics_n_stuff/PIFCamp_Kresnicka_25_v1.1.kicad_pcb (KiCad board)
At the start: 2 copper layers, 27 x 29 mm, 11 parts, among them J1 Conn_01x01_Pin, U1 ATtiny85-20P, U2 TSOP382xx

Commit message: panelized
Parts:
- BZ1: footprint Buzzer_Beeper:Buzzer_12x9.5RM7.6 -> Buzzer_Beeper:Buzzer_TDK_PS1240P02BT_D12.2mm_H6.5mm
- U1: footprint Package_DIP:DIP-8_W7.62mm_Socket -> Package_DIP:DIP-8_W7.62mm_LongPads
- moved BZ1 0.20 mm to (105.5, 118.5)
Routing:
- net GND: track 63.8 -> 69.1 mm
- net Net-(BZ1-+): track 17.6 -> 18.8 mm
Other:
- board size 27 x 29 mm -> 27 x 28.5 mm
- board text added: "Kresnička V1 PIFcamp 2025"
